Commit message: added and updated a lot

File: husky_description/urdf/husky.urdf.xacro (robot description, xacro)
@@ -22,8 +22,8 @@
 -->
 <robot name="husky" xmlns:xacro="http://ros.org/wiki/xacro">
-  <xacro:arg name="laser_enabled" default="false" />
+  <xacro:arg name="laser_enabled" default="true" />
   <xacro:arg name="laser_xyz" default="$(optenv HUSKY_LMS1XX_XYZ 0.2206 0.0 0.00635)" />
   <xacro:arg name="laser_rpy" default="$(optenv HUSKY_LMS1XX_RPY 0.0 0.0 0.0)" />
-  <xacro:arg name="kinect_enabled" default="false" />
+  <xacro:arg name="kinect_enabled" default="true" />
   <xacro:arg name="kinect_xyz" default="$(optenv HUSKY_KINECT_XYZ 0 0 0)" />
   <xacro:arg name="kinect_rpy" default="$(optenv HUSKY_KINECT_RPY 0 0.18 3.14)" />

File: husky_description/urdf/sensors/kinect.urdf.xacro (robot description, xacro)
@@ -1,5 +1,5 @@
 <?xml version="1.0"?>
 <root name="sensor_kinect" xmlns:xacro="http://ros.org/wiki/xacro">
-	<xacro:include filename="$(find jackal_description)/urdf/sensors/kinect_gazebo.xacro" />
+	<xacro:include filename="$(find husky_description)/urdf/sensors/kinect_gazebo.xacro" />
    	<!-- camera_name has to be unique! -->
 	<xacro:kinect_sensor link_name="camera_depth_frame" camera_name="camera1" frame_name="camera_depth_optical_frame"/>
@@ -40,5 +40,5 @@
 			 <origin xyz="0 0 0" rpy="0 0 ${M_PI/2}"/>
 				<geometry>
-				<mesh filename="package://jackal_description/urdf/sensors/kinect.dae"/>
+				<mesh filename="package://husky_description/urdf/sensors/kinect.dae"/>
 				</geometry>
 			</visual>

File: husky_description/urdf/sensors/kinect_gazebo.xacro (robot description, xacro)
@@ -2,5 +2,5 @@
 <root name="kinect_gazebo" xmlns:xacro="http://ros.org/wiki/xacro">
   <!-- Microsoft Kinect / ASUS Xtion PRO Live for simulation -->
-  <xacro:include filename="$(find jackal_description)/urdf/sensors/common_properties.urdf.xacro" />
+  <xacro:include filename="$(find husky_description)/urdf/sensors/common_properties.urdf.xacro" />
   <xacro:macro name="kinect_sensor" params="link_name camera_name frame_name">
     <gazebo reference="${link_name}">
